Commit message: Fixada a câmera

File: IBVS_ws/src/realsense_gazebo_plugin/urdf/rs200_simulation.xacro (robot description, xacro)
@@ -10,5 +10,5 @@
     <!-- Create camera instance -->
     <xacro:realsense-rs200 prefix="" parent="world">
-        <origin xyz="0 0 1.0" rpy="0 0 0" />
+        <origin xyz="-0.6 2.1 1.2" rpy="0 0.27 -0.85" />
     </xacro:realsense-rs200>
 </robot>
