Commit message: Fixed IBVS Launch

File: IBVS_ws/src/ibvs_projeto/urdf/apriltag.urdf (robot description, URDF)
Before this commit: robot april_tag, 1 links, 0 joints
Links:
- link simple_box_base_link: geometry collision box size=0.2 0.2 0.2; visual mesh filename=package://ibvs_projeto/urdf/tag0.dae

Commit message: IBVS Tag Wall e Apriltag Detection funcionando

File: IBVS_ws/src/ibvs_projeto/urdf/apriltag.urdf (robot description, URDF)
Before this commit: robot april_tag, 1 links, 0 joints
Links:
- link simple_box_base_link: geometry collision box size=0.4 0.6 0.6; visual mesh filename=package://ibvs_projeto/urdf/tag_wall.dae

Commit message: IBVS QUASE LA

File: IBVS_ws/src/ibvs_projeto/urdf/apriltag.urdf (robot description, URDF)
Before this commit: robot april_tag, 1 links, 0 joints
Links:
- link simple_box_base_link: geometry collision box size=0.4 1.2 1.2; visual mesh filename=package://ibvs_projeto/urdf/tag_wall.dae
